File: AE_ESP_board/AE_ESP_board.brd (EAGLE design)
At the start: 47 x 47 mm, 26 parts, among them CN1 SW_UART_IF, CN2 HW_UART_IF, CN3 POWER_IF, Q1 2N7000, Q2 2N7000, SW1 10-XX, U1 AE-ESP-WROOM-02, U2 M78AR033-0.5

Commit message: LEDを表面実装にする理由がないので、こちらもリード部品化 （ただし3mm砲弾型前提）
Parts:
- D1, D2, D3: value LED_0805 -> LED_3MM; device Parts:CHIPLED_0805 -> Parts:LED3MM
- moved R8 13.3 mm to (21.6, 27.9)
- moved D3 12.8 mm to (33.0, 29.2)
- moved R4 9.92 mm to (8.89, 27.9), turned to 0 degrees
- moved R6 7.41 mm to (21.6, 40.6)
- moved R7 7.41 mm to (21.6, 34.3)
- moved D2 6.48 mm to (33.0, 35.6)
- moved D1 6.48 mm to (33.0, 41.9)
- moved Q1 1.27 mm to (5.08, 22.9)
Connections:
- net 0V: now also D1.K, D2.K, D3.K; no longer D1.C, D2.C, D3.C
Changed lines of the file:
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@@
 <setting verticaltext="up"/>
 </settings>
-<grid distance="50" unitdist="mil" unit="mil" style="lines" multiple="1" display="yes" altdistance="0.025" altunitdist="inch" altunit="inch"/>
+<grid distance="0.05" unitdist="inch" unit="inch" style="lines" multiple="1" display="no" altdistance="0.025" altunitdist="inch" altunit="inch"/>
 <layers>
 <layer number="1" name="Top" color="4" fill="1" visible="yes" active="yes"/>
@@
 <text x="26.035" y="1.905" size="0.8128" layer="21">(PROG)</text>
 <text x="2.8575" y="10.795" size="0.8128" layer="21" rot="R90">(DATA)</text>
-<text x="36.83" y="39.6875" size="0.8128" layer="21" rot="R90">SERVER</text>
-<text x="36.83" y="26.3525" size="0.8128" layer="21" rot="R90">CONNECT</text>
-<text x="36.83" y="33.3375" size="0.8128" layer="21" rot="R90">HCHECK</text>
+<text x="36.83" y="26.9875" size="0.8128" layer="21" rot="R90">SERVER</text>
+<text x="36.83" y="32.7025" size="0.8128" layer="21" rot="R90">CONNECT</text>
+<text x="36.83" y="39.6875" size="0.8128" layer="21" rot="R90">HCHECK</text>
 </plain>
 <attributes>
@@
 <attribute name="VALUE" x="33.02" y="0.3175" size="1.27" layer="27"/>
 </element>
-<element name="D1" library="Parts" package="CHIPLED_0805" value="LED_0805" x="34.29" y="35.56" rot="R90"/>
-<element name="D2" library="Parts" package="CHIPLED_0805" value="LED_0805" x="34.29" y="29.21" rot="R90"/>
-<element name="D3" library="Parts" package="CHIPLED_0805" value="LED_0805" x="34.29" y="41.91" rot="R90"/>
+<element name="D1" library="Parts" package="LED3MM" value="LED_3MM" x="33.02" y="41.91" rot="R90"/>
+<element name="D2" library="Parts" package="LED3MM" value="LED_3MM" x="33.02" y="35.56" rot="R90"/>
+<element name="D3" library="Parts" package="LED3MM" value="LED_3MM" x="33.02" y="29.21" rot="R90"/>
 <element name="H1" library="Generic" package="3,2" value="MOUNT_HOLE_3.2" x="44" y="44"/>
 <element name="H2" library="Generic" package="3,2" value="MOUNT_HOLE_3.2" x="3" y="44"/>
@@
 <attribute name="VALUE" x="36.8935" y="19.05" size="0.7112" layer="27" ratio="10" rot="R90"/>
 </element>
-<element name="Q1" library="Parts" package="TO-92NL" value="2N7000" x="6.35" y="22.86" smashed="yes" rot="R270">
-<attribute name="NAME" x="4.1275" y="15.875" size="0.8128" layer="25" ratio="10"/>
-<attribute name="VALUE" x="3.3655" y="21.9075" size="0.8128" layer="27" ratio="10" rot="R270"/>
+<element name="Q1" library="Parts" package="TO-92NL" value="2N7000" x="5.08" y="22.86" smashed="yes" rot="R270">
+<attribute name="NAME" x="2.8575" y="17.145" size="0.8128" layer="25" ratio="10" rot="R90"/>
+<attribute name="VALUE" x="2.0955" y="21.9075" size="0.8128" layer="27" ratio="10" rot="R270"/>
 </element>
 <element name="Q2" library="Parts" package="TO-92NL" value="2N7000" x="29.21" y="11.43" rot="R180"/>
@@
 <attribute name="VALUE" x="24.13" y="20.32" size="0.8128" layer="27" ratio="10"/>
 </element>
-<element name="R4" library="Parts" package="RESISTOR_0204_200MIL" value="10k" x="2.54" y="20.32" rot="R90"/>
+<element name="R4" library="Parts" package="RESISTOR_0204_200MIL" value="10k" x="8.89" y="27.94"/>
 <element name="R5" library="Parts" package="RESISTOR_0204_200MIL" value="10k" x="26.67" y="15.24" smashed="yes">
 <attribute name="NAME" x="25.7175" y="14.9225" size="0.8128" layer="25" ratio="10"/>
 <attribute name="VALUE" x="24.13" y="12.7" size="0.8128" layer="27" ratio="10"/>
 </element>
-<element name="R6" library="Parts" package="RESISTOR_0204_200MIL" value="330" x="25.4" y="34.29" rot="R180"/>
-<element name="R7" library="Parts" package="RESISTOR_0204_200MIL" value="330" x="25.4" y="27.94" rot="R180"/>
-<element name="R8" library="Parts" package="RESISTOR_0204_200MIL" value="330" x="25.4" y="40.64" rot="R180"/>
+<element name="R6" library="Parts" package="RESISTOR_0204_200MIL" value="330" x="21.59" y="40.64" rot="R180"/>
+<element name="R7" library="Parts" package="RESISTOR_0204_200MIL" value="330" x="21.59" y="34.29" rot="R180"/>
+<element name="R8" library="Parts" package="RESISTOR_0204_200MIL" value="330" x="21.59" y="27.94" rot="R180"/>
 <element name="SW1" library="Parts" package="B3F-10XX" value="10-XX" x="39.37" y="36.83"/>
 <element name="U1" library="PartsForProto" package="DIL18_AE-ESP-WROOM-02" value="AE-ESP-WROOM-02" x="11.43" y="22.86" smashed="yes" rot="R270">
-<attribute name="NAME" x="6.89" y="25.2318" size="1.778" layer="25" ratio="10"/>
+<attribute name="NAME" x="13.875" y="23.9618" size="1.778" layer="25" ratio="10"/>
 <attribute name="VALUE" x="14.351" y="22.86" size="1.778" layer="27" ratio="10" rot="R270"/>
 </element>
@@
 <contactref element="U1" pad="5"/>
 <contactref element="JP1" pad="1"/>
-<contactref element="D1" pad="C"/>
-<contactref element="D2" pad="C"/>
+<contactref element="D1" pad="K"/>
+<contactref element="D2" pad="K"/>
 <contactref element="SW1" pad="4"/>
-<contactref element="D3" pad="C"/>
+<contactref element="D3" pad="K"/>
 <contactref element="U1" pad="18"/>
 <contactref element="U1" pad="13"/>
@@
 <vertex x="-2.54" y="-1.27"/>
 </polygon>
-<wire x1="34.29" y1="37.01" x2="34.29" y2="43.36" width="0" layer="19" extent="1-1"/>
-<wire x1="34.29" y1="30.66" x2="34.29" y2="37.01" width="0" layer="19" extent="1-1"/>
-<wire x1="34.29" y1="22.86" x2="34.29" y2="30.66" width="0" layer="19" extent="1-1"/>
 </signal>
 <signal name="+3V3">
@@
 <wire x1="11.43" y1="20.32" x2="26.67" y2="11.43" width="0" layer="19" extent="1-1"/>
 <wire x1="11.43" y1="22.86" x2="11.43" y2="20.32" width="0" layer="19" extent="1-1"/>
-<wire x1="6.35" y1="20.32" x2="11.43" y2="20.32" width="0" layer="19" extent="1-1"/>
-<wire x1="2.54" y1="22.86" x2="6.35" y2="20.32" width="0" layer="19" extent="1-1"/>
+<wire x1="11.43" y1="27.94" x2="11.43" y2="22.86" width="0" layer="19" extent="1-1"/>
+<wire x1="5.08" y1="20.32" x2="11.43" y2="20.32" width="0" layer="19" extent="1-1"/>
 </signal>
 <signal name="HW_UART_TXD">
@@
 <contactref element="U1" pad="10"/>
 <contactref element="R7" pad="2"/>
-<wire x1="19.05" y1="2.54" x2="22.86" y2="27.94" width="0" layer="19" extent="1-1"/>
+<wire x1="19.05" y1="2.54" x2="19.05" y2="34.29" width="0" layer="19" extent="1-1"/>
 </signal>
 <signal name="LED_HCHECK">
 <contactref element="U1" pad="7"/>
 <contactref element="R6" pad="2"/>
-<wire x1="11.43" y1="7.62" x2="22.86" y2="34.29" width="0" layer="19" extent="1-1"/>
+<wire x1="11.43" y1="7.62" x2="19.05" y2="40.64" width="0" layer="19" extent="1-1"/>
 </signal>
 <signal name="N$11">
 <contactref element="D2" pad="A"/>
 <contactref element="R7" pad="1"/>
-<wire x1="27.94" y1="27.94" x2="34.29" y2="27.76" width="0" layer="19" extent="1-1"/>
+<wire x1="24.13" y1="34.29" x2="33.02" y2="34.29" width="0" layer="19" extent="1-1"/>
 </signal>
 <signal name="N$12">
 <contactref element="D1" pad="A"/>
 <contactref element="R6" pad="1"/>
-<wire x1="27.94" y1="34.29" x2="34.29" y2="34.11" width="0" layer="19" extent="1-1"/>
+<wire x1="24.13" y1="40.64" x2="33.02" y2="40.64" width="0" layer="19" extent="1-1"/>
 </signal>
 <signal name="SW_UART_RXD_IN">
@@
 <contactref element="Q1" pad="3"/>
 <contactref element="R4" pad="1"/>
-<wire x1="6.35" y1="17.78" x2="11.43" y2="17.78" width="0" layer="19" extent="1-1"/>
-<wire x1="2.54" y1="17.78" x2="6.35" y2="17.78" width="0" layer="19" extent="1-1"/>
+<wire x1="5.08" y1="17.78" x2="6.35" y2="27.94" width="0" layer="19" extent="1-1"/>
+<wire x1="11.43" y1="17.78" x2="5.08" y2="17.78" width="0" layer="19" extent="1-1"/>
 </signal>
 <signal name="SW_UART_RXD">
 <contactref element="Q1" pad="1"/>
 <contactref element="CN1" pad="2"/>
-<wire x1="5.08" y1="11.43" x2="6.35" y2="22.86" width="0" layer="19" extent="1-1"/>
+<wire x1="5.08" y1="11.43" x2="5.08" y2="22.86" width="0" layer="19" extent="1-1"/>
 </signal>
 <signal name="N$1">
@@
 <contactref element="U1" pad="14"/>
 <contactref element="R8" pad="2"/>
-<wire x1="19.05" y1="12.7" x2="22.86" y2="40.64" width="0" layer="19" extent="1-1"/>
+<wire x1="19.05" y1="12.7" x2="19.05" y2="27.94" width="0" layer="19" extent="1-1"/>
 </signal>
 <signal name="N$5">
 <contactref element="R8" pad="1"/>
 <contactref element="D3" pad="A"/>
-<wire x1="27.94" y1="40.64" x2="34.29" y2="40.46" width="0" layer="19" extent="1-1"/>
+<wire x1="24.13" y1="27.94" x2="33.02" y2="27.94" width="0" layer="19" extent="1-1"/>
 </signal>
 <signal name="N$3">

Commit message: 配線を確定
Routing:
- net +3V3: track 0.00 -> 58.4 mm
- net N$9: track 0.00 -> 45.9 mm
- net N$10: track 0.00 -> 40.4 mm
- net LED_HCHECK: track 0.00 -> 39.2 mm, vias 0 -> 2
- net LED_CONNECTING: track 0.00 -> 37.1 mm, vias 0 -> 2
- net +12V: track 0.00 -> 26.0 mm
- net SW_UART_RXD_IN: track 0.00 -> 21.4 mm
- net N$4: track 0.00 -> 19.2 mm, vias 0 -> 2
- net N$2: track 0.00 -> 17.3 mm
- net SW_UART_RXD: track 0.00 -> 15.0 mm
- net N$7: track 0.00 -> 13.0 mm
- net N$5: track 0.00 -> 8.89 mm
- net N$12: track 0.00 -> 8.89 mm
- net N$11: track 0.00 -> 8.89 mm
- net N$3: track 0.00 -> 7.40 mm
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